File: RasberryBooster/RasberryBooster.kicad_pcb (KiCad board)
At the start: 2 copper layers, 18.6 x 29.2 mm, 14 parts, among them J1 Conn_01x02_Socket, J2 Capacitor, J3 Conn_01x02_Socket

Commit message: Finished PCB design
Parts:
- removed ISL91127IRAZ-T7A1: ~, BuckBoosterLibrary:ISL91127IRAZ-T7A
- added ?: , , F.Cu at (106.2, 111.3)
- added ?: , , F.Cu at (48.2, 88.3)
- added ?: , , F.Cu at (106.2, 88.3)
- added ?: , , F.Cu at (48.2, 111.3)
- added C10: C, Capacitor_SMD:C_0603_1608Metric, F.Cu at (57.4, 110.0)
- added C9: C, Capacitor_SMD:C_0603_1608Metric, F.Cu at (55.9, 110.0)
- added D2: LED, LED_SMD:LED_0603_1608Metric, F.Cu at (49.6, 92.4)
- added G***: LOGO, BuckBoosterLibrary:USNACrest, B.Cu at (88.0, 102.8)
- added ISL: ~, BuckBoosterLibrary:ISL91127IRAZ-T7A, F.Cu at (53.9, 106.1)
- added J4: USB_A, Connector_USB:USB_Micro-B_Molex-105017-0001, F.Cu at (47.4, 99.9)
- added R5: R, Resistor_SMD:R_0603_1608Metric, F.Cu at (49.6, 93.9)
- added R6: 1k, Resistor_SMD:R_0603_1608Metric, F.Cu at (59.9, 103.9)
- added R7: 2k, Resistor_SMD:R_0603_1608Metric, F.Cu at (58.9, 110.1)
- added U1: ATtiny85-20P, Package_DIP:DIP-8_W7.62mm, F.Cu at (52.4, 93.0)
- J1: value Conn_01x02_Socket -> Conn_02x20_Odd_Even; footprint Connector_PinHeader_2.54mm:PinHeader_1x02_P2.54mm_Horizontal -> Connector_PinHeader_2.54mm:PinHeader_2x20_P2.54mm_Vertical; moved to F.Cu
- J2: footprint Connector_JST:JST_ZE_B02B-ZESK-1D_1x02_P1.50mm_Vertical -> Connector_PinSocket_2.54mm:PinSocket_1x02_P2.54mm_Vertical
- J3: value Conn_01x02_Socket -> Conn_01x02; footprint Connector_PinHeader_2.54mm:PinHeader_1x02_P2.54mm_Horizontal -> Connector_PinSocket_2.54mm:PinSocket_1x02_P2.54mm_Vertical; moved to F.Cu
- moved J2 111.3 mm to (53.2, 113.3), turned to 90 degrees
- moved C3 110.5 mm to (52.8, 110.1), turned to -90 degrees
- moved R1 109.1 mm to (51.5, 103.0), turned to 180 degrees
- moved C4 107.2 mm to (54.3, 110.1), turned to -90 degrees
- moved J1 105.4 mm to (53.1, 89.6), turned to 90 degrees
- moved J3 104.3 mm to (48.6, 106.3), turned to -90 degrees
- moved C2 104.1 mm to (59.9, 106.9), turned to 90 degrees
- moved C6 101.8 mm to (54.6, 103.0), turned to 0 degrees
- moved C8 97.8 mm to (50.8, 105.2), turned to -90 degrees
- moved L1 95.2 mm to (57.6, 106.1), turned to -90 degrees
- moved C7 92.3 mm to (57.6, 103.0), turned to 0 degrees
- moved C1 89.7 mm to (67.0, 97.3), turned to 90 degrees
- moved C5 85.3 mm to (67.0, 109.0), turned to 90 degrees
Connections:
- net Net-(ISL91127IRAZ-T7A1-EN) renamed +5VA
- J1 pad 1: Earth -> unconnected-(J1-Pin_1-Pad1)
- J1 pad 2: +5V -> +5C
- J3 pad 1: +5C -> +5V
- L1 pad 1: Net-(ISL91127IRAZ-T7A1-LX1-Pad4) -> L1
- L1 pad 2: Net-(ISL91127IRAZ-T7A1-LX2-Pad1) -> L2
Routing:
- net +5C: track 17.6 -> 41.1 mm
- net GPIO: track 0.00 -> 9.78 mm
- net +5V: track 2.53 -> 10.1 mm
- net Earth: track 44.0 -> 47.8 mm, vias 0 -> 2
- net +5VA: track 23.7 -> 20.2 mm, vias 0 -> 1
- net Net-(ISL91127IRAZ-T7A1-LX1-Pad4): track 2.63 -> 0.00 mm
- net Net-(U1-AREF/PB0): track 0.00 -> 2.48 mm
- net Net-(ISL91127IRAZ-T7A1-LX2-Pad1): track 2.47 -> 0.00 mm
- net Net-(D2-K): track 0.00 -> 1.53 mm
- added copper zone on F.Cu, net +5C
- added copper zone on F.Cu, net +5VA
- added copper zone on F.Cu, net L1
- added copper zone on F.Cu, net L2
Other:
- board size 18.6 x 29.2 mm -> 65 x 30 mm
- board text added: "+"
- board text added: "-"
- board text added: "Board Corner Radius = 3mm All holes are M2.5"
- board text added: "Ignore the ghost right angle. I dont think it can hurt you"
- board text added: "Poker chip for reference"
- board text added: "Victor E. Zimmerman MIDN USN NASA Intern GSFC Raspberry Buckboost"
